File: Akashi-14.kicad_pcb (KiCad board)
At the start: 2 copper layers, 67.3 x 91.4 mm, 10 parts, among them J1 Conn_02x35_Odd_Even, J2 Conn_02x35_Odd_Even, J3 CONN_N7E50-Q516RB-50_3MM

Commit message: Add version number
Other:
- board text added: "V1.0.0 Compact Flash for Nucleo"
- board text removed: "Compact Flash for Nucleo"
Changed lines of the file:
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@@
     (effects (font (size 1 1) (thickness 0.2) bold) (justify left bottom))
   )
-  (gr_text "Compact Flash for Nucleo" (at 122.682 91.44) (layer "F.SilkS")
+  (gr_text "V1.0.0\nCompact Flash for Nucleo" (at 122.682 91.44) (layer "F.SilkS")
     (effects (font (size 1 1) (thickness 0.15)) (justify left bottom))
   )
